File: phone/phone_pcb/phone_pcb.kicad_sch (KiCad schematic)
At the start: 24 parts, among them J1 Raspberry_Pi_2_3, J2 RJ11, U1 Ag1171S, X1 ASE-24.576MHz

Commit message: Design the PCB!
Parts:
- added C10, C4, C6, C8: 10u, Capacitor_Tantalum_SMD:CP_EIA-3216-18_Kemet-A, symbol Device:C_Polarized_US
- C1: value 100n -> 10n; footprint (none) -> Capacitor_SMD:C_0402_1005Metric
- C11, C13, C2, C3, C5, C7, C9: footprint (none) -> Capacitor_SMD:C_0402_1005Metric
- C12: footprint (none) -> Capacitor_THT:C_Radial_D6.3mm_H7.0mm_P2.50mm
- J2: footprint (none) -> Connector_RJ:RJ11_Ckmtw_A800_Horizontal
- R1: footprint (none) -> Resistor_SMD:R_0402_1005Metric
- R2: footprint (none) -> Resistor_SMD:R_0805_2012Metric
- TP1, TP2, TP3, TP4, TP5, TP6, TP7, TP8: footprint (none) -> TestPoint:TestPoint_THTPad_D2.0mm_Drill1.0mm
- U1: footprint Connector_PinSocket_2.54mm:PinSocket_1x18_P2.54mm_Vertical -> Connector_PinHeader_2.54mm:PinHeader_1x7+7_P2.54mm_Vertical
Connections:
- net +3.3V: now also C8.1
- net +5V: now also C10.1
- net GND: now also C10.2, C4.2, C6.2, C8.2
- net at C7.2, PCM1.3 (V_{REF1}): now also C6.1
- net at C5.2, PCM1.4 (V_{REF2}), R1.2: now also C4.1
Other:
- moved on the sheet: C7, R1, TP8

Commit message: Do some DNPs
Parts:
- C1: LCSC (none) -> C15195
- C10, C4, C6, C8: LCSC (none) -> C7171
- C11, C13, C5, C7, C9: LCSC (none) -> C1525
- C12, TP1, TP2, TP3, TP4, TP5, TP6, TP7, TP8, U1: now not fitted
- C2, C3: LCSC (none) -> C52923
- J1: LCSC (none) -> C25503128
- J2: LCSC (none) -> C189748
- PCM1: LCSC (none) -> C2866894
- R1: LCSC (none) -> C11702
- R2: LCSC (none) -> C4328
- X1: LCSC (none) -> C437128
