File: phone/phone_pcb/_autosave-phone_pcb.kicad_sch (KiCad schematic)
At the start: 29 parts, among them J1 Raspberry_Pi_2_3, J2 RJ11, U1 Ag1171S, X1 ASE-24.576MHz

Commit message: Rev0.1 of PCB :D
Parts:
- J1: LCSC C25503128 -> C2685115
Changed lines of the file:
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@@
 			)
 		)
-		(property "LCSC" "C25503128"
+		(property "LCSC" "C2685115"
 			(at 50.8 83.82 0)
 			(effects
